File: 555re4.brd (EAGLE design)
At the start: 142.2 x 142.2 mm, 69 parts, among them IC1 4011D

Commit message: 2
Parts:
- added R4, R5: 2*2, rcl:M0805
- LED1, LED10, LED11, LED12, LED13, LED14, LED15, LED16, LED17, LED18, LED19, LED2, LED20, LED21, LED22, LED23, LED24, LED25, LED27, LED28, LED29, LED3, LED30, LED31, LED32, LED33, LED34, LED35, LED36, LED37, LED38, LED39, LED4, LED40, LED41, LED42, LED43, LED44, LED45, LED46, LED47, LED48, LED49, LED50, LED51, LED52, LED53, LED54, LED55, LED56, LED6, LED7, LED8, LED9: device SparkFun-LED:LED5MM-KIT -> SparkFun-LED:LED3MM
- LED26: device SparkFun-LED:LED5MM-KIT -> SparkFun-LED:LED3MM-NS
- R1: value 2*2 -> 1k
- R3: value 1k -> 2*2; device rcl:0207/10 -> rcl:M0805
- moved IC1 115.1 mm to (82.5, 95.9)
- moved R3 68.3 mm to (155.9, 106.5), flipped to the bottom, turned to 247.5 degrees
- moved R1 58.4 mm to (94.6, 76.2), turned to 270 degrees
- moved LED56 30.6 mm to (163.8, 87.6)
- moved LED48 25.5 mm to (159.4, 87.6)
- moved LED40 20.4 mm to (154.9, 87.6)
- moved LED32 15.3 mm to (150.5, 87.6)
- moved LED52 12.7 mm to (39.4, 87.6)
- moved C2 11.7 mm to (150.2, 110.3), turned to 202.5 degrees
- moved LED49 11.7 mm to (146.1, 43.2), turned to 225 degrees
- moved LED51 11.7 mm to (57.1, 43.2)
- moved LED53 11.7 mm to (57.1, 132.1), turned to 45 degrees
- moved LED55 11.7 mm to (146.1, 132.1), turned to 315 degrees
- moved LED44 10.8 mm to (43.8, 87.6)
- moved C1 10.2 mm to (142.5, 102.3), turned to 292.5 degrees
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Connections:
- new net N$66: R3.1, R5.2
- new net N$67: DA1.9
- new net N$68: DA1.10
- new net N$69: DA1.11
- new net N$70: DA1.12
- new net N$71: DA1.13
- new net N$72: DA1.14
- new net N$73: DA1.15
- new net N$74: DA1.16
- net GND: now also R1.2; no longer R3.2
- net N$15: now also R3.2, R4.2; no longer R1.2
- net N$19: now also R1.1; no longer R3.1
- net VCC: now also R4.1, R5.1; no longer R1.1
Routing:
- net N$6: track 21.7 -> 23.9 mm
- net N$9: track 20.6 -> 19.4 mm
- net N$7: track 21.7 -> 22.3 mm
Other:
- board size 142.2 x 142.2 mm -> 132.1 x 132.1 mm
