File: 555re4.sch (EAGLE design)
At the start: 69 parts, among them IC1 4011D

Commit message: 2
Parts:
- added R4, R5: 2*2, rcl:R-EU_M0805
- LED1, LED10, LED11, LED12, LED13, LED14, LED15, LED16, LED17, LED18, LED19, LED2, LED20, LED21, LED22, LED23, LED24, LED25, LED27, LED28, LED29, LED3, LED30, LED31, LED32, LED33, LED34, LED35, LED36, LED37, LED38, LED39, LED4, LED40, LED41, LED42, LED43, LED44, LED45, LED46, LED47, LED48, LED49, LED50, LED51, LED52, LED53, LED54, LED55, LED56, LED6, LED7, LED8, LED9: device SparkFun-LED:LED5MM-KIT -> SparkFun-LED:LED3MM
- LED26: device SparkFun-LED:LED5MM-KIT -> SparkFun-LED:LED-3MM-NO_SILK
- R1: value 2*2 -> 1k
- R3: value 1k -> 2*2; device rcl:R-EU_0207/10 -> rcl:R-EU_M0805
Connections:
- new net N$66: R3.1, R5.2
- new net N$67: DA1.CD+
- new net N$68: DA1.O7
- new net N$69: DA1.O6
- new net N$70: DA1.O5
- new net N$71: DA1.O4
- new net N$72: DA1.O3
- new net N$73: DA1.O2
- new net N$74: DA1.O1
- net GND: now also R1.2; no longer R3.2
- net N$15: now also R3.2, R4.2; no longer R1.2
- net N$19: now also R1.1; no longer R3.1
- net VCC: now also R4.1, R5.1; no longer R1.1
Other:
- moved on the sheet: LED1, LED2, LED3, LED4, LED5, LED6, LED7, LED8, R1, R3
